File: v1/kicad/v1.kicad_sch (KiCad schematic)
At the start: 3 parts, among them U1 RB, U2 RC, U3 RD

Commit message: partial
Parts:
- added U10: LNCPU FLAGS Register, lncpu:LNCPU FLAGS Register, symbol lncpu:LNCPU_FLAGS_Register
- added U11: LNCPU RAM, lncpu:LNCPU_RAM, symbol lncpu:LNCPU_RAM
- added U12: LNCPU ROM, symbol lncpu:LNCPU_ROM
- added U5: LNCPU ALU Operand Selector, lncpu:LNCPU_Alu_Operand_Selector, symbol lncpu:LNCPU_Alu_Operand_Selector
- added U8: LNCPU ALU, lncpu:LNCPU_ALU, symbol lncpu:LNCPU_ALU
- added U9: RA, lncpu:LNCPU_Shift_Register, symbol lncpu:LNCPU_Shift_Register
Connections:
- net DBUS0: now also U10.4 (DBUS_{0}), U11.19 (DBUS_{0}), U12.19 (DBUS_{0}), U8.4 (DBUS_{0}), U9.4 (DBUS_{0})
- net DBUS1: now also U10.6 (DBUS_{1}), U11.21 (DBUS_{1}), U12.21 (DBUS_{1}), U8.6 (DBUS_{1}), U9.6 (DBUS_{1})
- net DBUS2: now also U10.8 (DBUS_{2}), U11.23 (DBUS_{2}), U12.23 (DBUS_{2}), U8.8 (DBUS_{2}), U9.8 (DBUS_{2})
- net DBUS3: now also U10.10 (DBUS_{3}), U11.25 (DBUS_{3}), U12.25 (DBUS_{3}), U8.10 (DBUS_{3}), U9.10 (DBUS_{3})
- net DBUS4: now also U10.12 (DBUS_{4}), U11.27 (DBUS_{4}), U12.27 (DBUS_{4}), U8.12 (DBUS_{4}), U9.12 (DBUS_{4})
- net DBUS5: now also U10.14 (DBUS_{5}), U11.29 (DBUS_{5}), U12.29 (DBUS_{5}), U8.14 (DBUS_{5}), U9.14 (DBUS_{5})
- net DBUS6: now also U10.16 (DBUS_{6}), U11.31 (DBUS_{6}), U12.31 (DBUS_{6}), U8.16 (DBUS_{6}), U9.16 (DBUS_{6})
- net DBUS7: now also U10.18 (DBUS_{7}), U11.33 (DBUS_{7}), U12.33 (DBUS_{7}), U8.18 (DBUS_{7}), U9.18 (DBUS_{7})
- net GND: now also U10.1 (GND), U10.17 (GND), U10.20 (GND), U10.22 (GND), U11.1 (GND), U11.37 (GND), U11.38 (GND), U11.39 (GND), U12.1 (GND), U12.37 (GND), U12.38 (GND), U12.39 (GND), U5.1 (GND), U5.10 (GND), U5.12 (GND), U5.14 (GND), U8.1 (GND), U8.17 (GND), U8.20 (GND), U8.22 (GND), U9.1 (GND), U9.17 (GND), U9.20 (GND), U9.22 (GND), U9.23 (CLK2)
- net RST: now also U9.13 (CTRL_{5})
- net VCC: now also U10.2 (VCC), U10.24 (VCC), U11.2 (VCC), U11.40 (VCC), U12.2 (VCC), U12.40 (VCC), U5.16 (VCC), U5.2 (VCC), U8.2 (VCC), U8.24 (VCC), U9.2 (VCC), U9.24 (VCC)
- net at U1.21 (CLK1): now also U9.15 (CTRL_{6})
- net at U1.7 (~{R_{out}}): now also U9.11 (CTRL_{4})
- removed net PHI_{2}: U1.3 (~{R_{en}}), U2.3 (~{R_{en}}), U3.3 (~{R_{en}})
- new net: U10.13 (ALU_{Cin}), U8.13 (C_{out})
- new net ABUS0: U11.4 (ABUS_{0}), U12.4 (ABUS_{0})
- new net ABUS1: U11.6 (ABUS_{1}), U12.6 (ABUS_{1})
- new net ABUS10: U11.24 (ABUS_{10}), U12.24 (ABUS_{10})
- new net ABUS11: U11.26 (ABUS_{11}), U12.26 (ABUS_{11})
- new net ABUS12: U11.28 (ABUS_{12}), U12.28 (ABUS_{12})
- new net ABUS2: U11.8 (ABUS_{2}), U12.8 (ABUS_{2})
- new net ABUS3: U11.10 (ABUS_{3}), U12.10 (ABUS_{3})
- new net ABUS4: U11.12 (ABUS_{4}), U12.12 (ABUS_{4})
- new net ABUS5: U11.14 (ABUS_{5}), U12.14 (ABUS_{5})
- new net ABUS6: U11.16 (ABUS_{6}), U12.16 (ABUS_{6})
- new net ABUS7: U11.18 (ABUS_{7}), U12.18 (ABUS_{7})
- new net ABUS8: U11.20 (ABUS_{8}), U12.20 (ABUS_{8})
- new net ABUS9: U11.22 (ABUS_{9}), U12.22 (ABUS_{9})
Other:
- added sheet AddressDecoder (AddressDecoder.kicad_sch)
- added sheet DeviceOEPhaseSelector (DeviceOEPhaseSelector.kicad_sch)
- moved on the sheet: U1, U2, U3
