File: v1/kicad/control_unit/control_unit.kicad_sch (KiCad schematic)
At the start: 2 parts, among them IC1 AT28C64B-15PU, J1 LNCPU_Control_Unit_Connector

Commit message: control unit
Parts:
- added IC2, IC3, IC4, IC5, IC6: AT28C64B-15PU, DIP1556W56P254L3702H483Q28N, symbol SamacSys_Parts:AT28C64B-15PU
- added J2: OP_{out}, Connector_PinSocket_2.54mm:PinSocket_1x08_P2.54mm_Vertical, symbol lncpu:LNCPU_DBUS_Socket
- added R1, R2, R3, R4, R5, R6, R7, R8: 4.7k, symbol Device:R
- added SW1: SW_DIP_x08, symbol Switch:SW_DIP_x08
- added U1, U2: 74LS155, Package_DIP:DIP-16_W7.62mm_LongPads, symbol 74xx:74LS155
- added U10, U9: 74LS157, Package_DIP:DIP-16_W7.62mm_LongPads, symbol 74xx:74LS157
- added U11, U12: 74HCT173, Package_DIP:DIP-16_W7.62mm_LongPads, symbol 74xx:74HCT173
- added U13: 74LS163, Package_DIP:DIP-16_W7.62mm_LongPads, symbol 74xx:74LS163
- added U14: 74LS32, Package_DIP:DIP-14_W7.62mm_LongPads, symbol 74xx:74LS32
- added U3, U4, U5, U6, U7, U8: 74HCT244, Package_DIP:DIP-20_W7.62mm_LongPads, symbol 74xx:74LS244
Connections:
- net ROM_{addr}12 is gone; now on net GND: IC1.2 (A12)
- net CLK: now also U11.7 (Cp), U12.7 (Cp), U13.2 (CP)
- net GND: now also IC1.14 (GND), IC1.20 (~{CE}), IC1.22 (~{OE}), IC2.14 (GND), IC2.2 (A12), IC2.20 (~{CE}), IC2.22 (~{OE}), IC3.14 (GND), IC3.2 (A12), IC3.20 (~{CE}), IC3.22 (~{OE}), IC4.14 (GND), IC4.2 (A12), IC4.20 (~{CE}), IC4.22 (~{OE}), IC5.14 (GND), IC5.2 (A12), IC5.20 (~{CE}), IC5.22 (~{OE}), IC6.14 (GND), IC6.2 (A12), IC6.20 (~{CE}), IC6.22 (~{OE}), R1.2, R2.2, R3.2, R4.2, R5.2, R6.2, R7.2, R8.2, U1.1 (Ea1), U1.14 (Eb1), U1.15 (Eb2), U1.8 (GND), U10.15 (E), U10.8 (GND), U13.8 (GND), U14.10, U14.12, U14.13, U14.4, U14.5, U14.7 (GND), U14.9, U2.1 (Ea1), U2.14 (Eb1), U2.15 (Eb2), U2.8 (GND), U3.1 (OEa), U3.10 (GND), U3.19 (OEb), U4.1 (OEa), U4.10 (GND), U4.19 (OEb), U5.1 (OEa), U5.10 (GND), U5.19 (OEb), U6.1 (OEa), U6.10 (GND), U6.19 (OEb), U7.1 (OEa), U7.10 (GND), U7.19 (OEb), U8.1 (OEa), U8.10 (GND), U8.19 (OEb), U9.15 (E), U9.8 (GND)
- net ROM_{addr}0: now also IC2.10 (A0), IC3.10 (A0), IC4.10 (A0), IC5.10 (A0), IC6.10 (A0), U13.14 (Q0)
- net ROM_{addr}1: now also IC2.9 (A1), IC3.9 (A1), IC4.9 (A1), IC5.9 (A1), IC6.9 (A1), U13.13 (Q1)
- net ROM_{addr}10: now also IC2.21 (A10), IC3.21 (A10), IC4.21 (A10), IC5.21 (A10), IC6.21 (A10), U10.9 (Zc)
- net ROM_{addr}11: now also IC2.23 (A11), IC3.23 (A11), IC4.23 (A11), IC5.23 (A11), IC6.23 (A11), U10.12 (Zd)
- net ROM_{addr}2: now also IC2.8 (A2), IC3.8 (A2), IC4.8 (A2), IC5.8 (A2), IC6.8 (A2), U13.12 (Q2)
- net ROM_{addr}3: now also IC2.7 (A3), IC3.7 (A3), IC4.7 (A3), IC5.7 (A3), IC6.7 (A3), U13.11 (Q3)
- net ROM_{addr}4: now also IC2.6 (A4), IC3.6 (A4), IC4.6 (A4), IC5.6 (A4), IC6.6 (A4), U9.4 (Za)
- net ROM_{addr}5: now also IC2.5 (A5), IC3.5 (A5), IC4.5 (A5), IC5.5 (A5), IC6.5 (A5)
- net ROM_{addr}6: now also IC2.4 (A6), IC3.4 (A6), IC4.4 (A6), IC5.4 (A6), IC6.4 (A6), U9.7 (Zb), U9.9 (Zc)
- net ROM_{addr}7: now also IC2.3 (A7), IC3.3 (A7), IC4.3 (A7), IC5.3 (A7), IC6.3 (A7), U9.12 (Zd)
- net ROM_{addr}8: now also IC2.25 (A8), IC3.25 (A8), IC4.25 (A8), IC5.25 (A8), IC6.25 (A8), U10.4 (Za)
- net ROM_{addr}9: now also IC2.24 (A9), IC3.24 (A9), IC4.24 (A9), IC5.24 (A9), IC6.24 (A9), U10.7 (Zb)
- net VCC: now also IC1.27 (~{WE}), IC1.28 (VCC), IC2.27 (~{WE}), IC2.28 (VCC), IC3.27 (~{WE}), IC3.28 (VCC), IC4.27 (~{WE}), IC4.28 (VCC), IC5.27 (~{WE}), IC5.28 (VCC), IC6.27 (~{WE}), IC6.28 (VCC), SW1.1, SW1.2, SW1.3, SW1.4, SW1.5, SW1.6, SW1.7, SW1.8, U1.16 (VCC), U1.2 (Ea2), U10.16 (VCC), U13.10 (CET), U13.16 (VCC), U13.3 (D0), U13.4 (D1), U13.5 (D2), U13.6 (D3), U13.7 (CEP), U13.9 (~{PE}), U14.14 (VCC), U2.16 (VCC), U2.2 (Ea2), U3.20 (VCC), U4.20 (VCC), U5.20 (VCC), U6.20 (VCC), U7.20 (VCC), U8.20 (VCC), U9.16 (VCC)
- net ~{IRQ}: now also U14.2
- net at J1.10 (CSPC_{up}): now also U6.12 (O3a)
- net at J1.11 (~{RC_{in}}): now also U4.9 (O0b)
- net at J1.12 (J_{mode0}): now also U6.9 (O0b)
- net at J1.13 (~{RD_{in}}): now also U4.7 (O1b)
- net at J1.14 (J_{mode1}): now also U6.7 (O1b)
- net at J1.15 (~{RT_{in}}): now also U4.5 (O2b)
- net at J1.16 (ADDR_{sel0}): now also U6.5 (O2b)
- net at J1.17 (~{RT_{out}}): now also U4.3 (O3b)
- net at J1.18 (ADDR_{sel1}): now also U6.3 (O3b)
- net at J1.19 (~{RB_{out}}): now also U3.18 (O0a)
- net at J1.20 (~{FETCH}): now also U7.18 (O0a)
- net at J1.21 (~{RC_{out}}): now also U3.16 (O1a)
- net at J1.22 (~{DL_{out}}): now also U7.16 (O1a)
- net at J1.23 (~{RD_{out}}): now also U3.14 (O2a)
- net at J1.24 (~{IVH_{out}}): now also U7.14 (O2a)
- net at J1.26 (~{IVL_{out}}): now also U7.12 (O3a)
- net at J1.28 (~{DS_{in}}): now also U7.9 (O0b)
- net at J1.29 (SP_{S0}): now also U3.7 (O1b)
- net at J1.30 (~{DS_{out}}): now also U7.7 (O1b)
- net at J1.31 (SP_{S1}): now also U3.5 (O2b)
- net at J1.32 (~{HLT}): now also U7.5 (O2b)
- net at J1.33 (~{SP_{out}}): now also U3.3 (O3b)
- net at J1.35 (~{ABL_{in}}): now also U5.18 (O0a)
- net at J1.36 (~{FLAGS_{out}}): now also U7.3 (O3b)
- net at J1.37 (~{ABH_{in}}): now also U5.16 (O1a)
- net at J1.38 (FLAGS_{sel1}): now also U8.18 (O0a)
- net at J1.39 (~{DEV_{in}}): now also U5.14 (O2a)
- net at J1.4 (~{CS_{in}}): now also U6.18 (O0a)
- net at J1.40 (FLAGS_{sel0}): now also U8.16 (O1a)
- net at J1.41 (~{DEV_{out}}): now also U5.12 (O3a)
- net at J1.42 (OP_{sel2}): now also U8.14 (O2a)
- net at J1.43 (X_{sel0}): now also U5.9 (O0b)
- net at J1.44 (OP_{sel1}): now also U8.12 (O3a)
- net at J1.45 (X_{sel1}): now also U5.7 (O1b)
- net at J1.46 (OP_{sel0}): now also U8.9 (O0b)
- net at J1.47 (X_{sel2}): now also U5.5 (O2b)
- net at J1.49 (Y_{sel0}): now also U5.3 (O3b)
- net at J1.6 (~{PC_{in}}): now also U6.16 (O1a)
- net at J1.8 (~{CSPC_{ct}}): now also U6.14 (O2a)
- net at J1.9 (~{RB_{in}}): now also U4.12 (O3a)
- net RA_{S0}: no longer names the net of J1.3 (RA_{S0})
- net RA_{S0}: now also U4.18 (O0a); no longer IC1.11 (I/O0)
- net RA_{S1}: no longer names the net of J1.5 (RA_{S1})
- net RA_{S1}: now also U4.16 (O1a); no longer IC1.12 (I/O1)
- net REGin_{sel0}: no longer names the net of IC1.15 (I/O3)
- net REGin_{sel0}: now also U1.13 (A0)
- net REGin_{sel1}: no longer names the net of IC1.16 (I/O4)
- net REGin_{sel1}: now also U1.3 (A1)
- net REGout_{sel0}: no longer names the net of IC1.17 (I/O5)
- net REGout_{sel0}: now also U2.13 (A0)
- net REGout_{sel1}: no longer names the net of IC1.18 (I/O6)
- net REGout_{sel1}: now also U2.3 (A1)
- net ~{RA_{out}}: no longer names the net of J1.7 (~{RA_{out}})
- net ~{RA_{out}}: now also U4.14 (O2a); no longer IC1.13 (I/O2)
- net ~{SS_{in}}: no longer names the net of J1.25 (~{SS_{in}})
- net ~{SS_{in}}: now also U3.12 (O3a); no longer IC1.19 (I/O7)
- net ~{SS_{out}}: no longer names the net of J1.27 (~{SS_{out}})
- net ~{SS_{out}}: now also U3.9 (O0b)
- new net: U1.11 (Q2b), U4.11 (I0b)
- new net: U1.12 (Q3b), U4.13 (I1b)
- new net: U2.10 (Q1b), U4.15 (I2b)
- new net: U2.11 (Q2b), U4.17 (I3b)
- new net: IC1.11 (I/O0), U4.2 (I0a)
- new net: IC1.12 (I/O1), U4.4 (I1a)
- new net: IC1.13 (I/O2), U4.6 (I2a)
- new net: U1.10 (Q1b), U4.8 (I3a)
- new net: IC5.11 (I/O0), U7.4 (I1a)
- new net: IC5.12 (I/O1), U7.6 (I2a)
- new net: IC5.13 (I/O2), U7.8 (I3a)
- new net: IC5.15 (I/O3), U7.11 (I0b)
- new net: IC5.16 (I/O4), U7.13 (I1b)
- new net: IC5.17 (I/O5), U7.15 (I2b)
- new net: IC5.18 (I/O6), U7.17 (I3b)
- new net: IC5.19 (I/O7), U8.2 (I0a)
- new net: IC4.19 (I/O7), U7.2 (I0a)
- new net: U2.12 (Q3b), U3.2 (I0a)
- new net: IC4.11 (I/O0), U6.4 (I1a)
- new net: IC4.12 (I/O1), U6.6 (I2a)
- new net: IC4.13 (I/O2), U6.8 (I3a)
- new net: IC4.15 (I/O3), U6.11 (I0b)
- new net: IC4.16 (I/O4), U6.13 (I1b)
- new net: IC4.17 (I/O5), U6.15 (I2b)
- new net: IC4.18 (I/O6), U6.17 (I3b)
- new net: IC3.15 (I/O3), U5.11 (I0b)
- new net: IC3.16 (I/O4), U5.13 (I1b)
- new net: IC3.17 (I/O5), U5.15 (I2b)
- new net: IC3.18 (I/O6), U5.17 (I3b)
- new net: IC2.19 (I/O7), U5.2 (I0a)
- new net: IC3.11 (I/O0), U5.4 (I1a)
- new net: IC3.12 (I/O1), U5.6 (I2a)
- new net: IC3.13 (I/O2), U5.8 (I3a)
- new net: R3.1, SW1.14, U9.11 (I0c)
- new net: R6.1, SW1.11, U10.5 (I0b)
- new net: IC6.11 (I/O0), U8.4 (I1a)
- new net: IC6.12 (I/O1), U8.6 (I2a)
- new net: IC6.13 (I/O2), U8.8 (I3a)
- new net: IC6.15 (I/O3), U8.11 (I0b)
- new net: IC6.16 (I/O4), U8.13 (I1b)
- new net: IC6.17 (I/O5), U8.15 (I2b)
- new net: IC6.18 (I/O6), U8.17 (I3b)
- new net: U10.1 (S), U14.3, U9.1 (S)
- new net: U11.5 (Q2), U9.10 (I1c)
- new net: U11.6 (Q3), U9.13 (I1d)
- new net: R4.1, SW1.13, U9.14 (I0d)
- new net: R1.1, SW1.16, U9.2 (I0a)
- new net: U11.3 (Q0), U9.3 (I1a)
- new net: R2.1, SW1.15, U9.5 (I0b)
- new net: U11.4 (Q1), U9.6 (I1b)
- new net: R7.1, SW1.10, U10.11 (I0c)
- new net: IC2.15 (I/O3), U3.11 (I0b)
- new net: IC2.16 (I/O4), U3.13 (I1b)
- new net: IC2.17 (I/O5), U3.15 (I2b)
- new net: IC2.18 (I/O6), U3.17 (I3b)
- new net: IC2.11 (I/O0), U3.4 (I1a)
- new net: IC2.12 (I/O1), U3.6 (I2a)
- new net: IC2.13 (I/O2), U3.8 (I3a)
- new net: IC3.19 (I/O7), U6.2 (I0a)
- new net: R8.1, SW1.9, U10.14 (I0d)
- new net: J2.1 (D0), U11.14 (D0)
- new net: J2.2 (D1), U11.13 (D1)
- new net: J2.3 (D2), U11.12 (D2)
- new net: J2.4 (D3), U11.11 (D3)
- new net: J2.5 (D4), U12.14 (D0)
- new net: J2.6 (D5), U12.13 (D1)
- new net: J2.7 (D6), U12.12 (D2)
- new net: J2.8 (D7), U12.11 (D3)
- new net: U11.1 (Oe1), U11.2 (Oe2), U11.8 (GND), U12.10 (E2), U12.8 (GND), U12.9 (E1)
- new net: U11.15 (Mr), U12.15 (Mr)
- new net: U11.16 (VCC), U12.16 (VCC)
- new net: U10.3 (I1a), U12.3 (Q0)
- new net: U10.6 (I1b), U12.4 (Q1)
- new net: U10.10 (I1c), U12.5 (Q2)
- new net: U10.13 (I1d), U12.6 (Q3)
- new net: R5.1, SW1.12, U10.2 (I0a)
- new net I: U14.1
- new net ~{PASS}: U11.10 (E2), U11.9 (E1), U12.1 (Oe1), U12.2 (Oe2), U13.1 (~{MR}), U8.7 (O1b)
- no-connect marks 0 -> 14
Other:
- moved on the sheet: IC1, J1
