File: v1/kicad/alu/alu/alu.kicad_pcb (KiCad board)
At the start: 2 copper layers, 223 x 137 mm, 23 parts, among them J1 LNCPU_Type_A_connector,_male,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, J2 X_{in}, J3 Y_{in}, J4 ALU_C_flag_info_socket, U1 74LS138, U10 74HC86, U11 74HC86, U12 74LS244, U13 74AHC04, U14 74AHC04, U15 74LS83, U16 74HC86, U17 74HC86, U18 74LS244, U19 74LS08, U2 74LS83, U3 74LS32, U4 74LS32, U5 74LS244, U6 74LS244, U7 74LS08, U8 74LS08, U9 74LS244

Commit message: partial
Parts:
- removed J1: LNCPU_Type_A_connector,_male,_active_high_reset, LNCPU:LNCPU_TYPE_A_MALE
- removed J4: ALU_C_flag_info_socket, Connector_PinSocket_2.54mm:PinSocket_1x02_P2.54mm_Vertical
- added U20: LNCPU Type B Connector, lncpu:LNCPU_Type_B_Header, F.Cu at (170.6, 54.0)
- added U21: 74HC86, Package_DIP:DIP-14_W7.62mm_LongPads, F.Cu at (127.2, 54.4)
- U1, U15, U2: footprint Package_DIP:DIP-16_W7.62mm -> Package_DIP:DIP-16_W7.62mm_LongPads
- U10, U11, U13, U14, U16, U17, U19, U3, U4, U7, U8: footprint Package_DIP:DIP-14_W7.62mm -> Package_DIP:DIP-14_W7.62mm_LongPads
- U12, U18, U5, U6, U9: footprint Package_DIP:DIP-20_W7.62mm -> Package_DIP:DIP-20_W7.62mm_LongPads
- moved U1 164.7 mm to (226.3, 59.5)
- moved J3 140.4 mm to (146.1, 171.0)
- moved J2 135.0 mm to (223.6, 170.0), turned to -90 degrees
- moved U16 130.5 mm to (54.4, 143.3), turned to 0 degrees
- moved U12 124.8 mm to (317.9, 80.5), turned to -90 degrees
- moved U17 108.0 mm to (80.0, 142.8), turned to 0 degrees
- moved U5 98.6 mm to (144.9, 80.2), turned to -90 degrees
- moved U14 85.6 mm to (301.9, 107.8), turned to 0 degrees
- moved U2 84.4 mm to (62.0, 127.0), turned to 180 degrees
- moved U6 81.3 mm to (198.8, 80.5), turned to -90 degrees
- moved U13 72.4 mm to (300.4, 144.3), turned to 0 degrees
- moved U9 70.2 mm to (258.4, 80.5), turned to -90 degrees
- moved U15 54.8 mm to (87.1, 127.9), turned to 180 degrees
- moved U3 54.7 mm to (129.2, 111.9)
- moved U19 46.4 mm to (77.7, 54.4)
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Connections:
- U14 pad 8: Net-(J4-SUB) -> Net-(U14-Pad8)
- U14 pad 9: /~{EN2} -> Net-(U18-OEa)
- U19 pad 1: GND -> Net-(U19-Pad1)
- U19 pad 2: GND -> Net-(U14-Pad8)
- U19 pad 3: unconnected-(U19-Pad3) -> C_{out}
Routing:
- net GND: track 0.00 -> 1154.4 mm, vias 0 -> 16
- net VCC: track 0.00 -> 916.3 mm, vias 0 -> 20
- net Net-(U15-C0): track 0.00 -> 453.7 mm, vias 0 -> 7
- net Net-(U18-OEa): track 0.00 -> 436.6 mm, vias 0 -> 6
- net /X4: track 0.00 -> 430.0 mm, vias 0 -> 9
- net /Y7: track 0.00 -> 419.1 mm, vias 0 -> 6
- net /D2: track 0.00 -> 410.9 mm, vias 0 -> 9
- net /X7: track 0.00 -> 410.8 mm, vias 0 -> 4
- net /X6: track 0.00 -> 409.3 mm, vias 0 -> 9
- net ~{ALU_{out}}: track 0.00 -> 397.6 mm, vias 0 -> 6
- net /X3: track 0.00 -> 394.6 mm, vias 0 -> 4
- net /D6: track 0.00 -> 393.9 mm, vias 0 -> 12
- net /X5: track 0.00 -> 391.1 mm, vias 0 -> 8
- net /D7: track 0.00 -> 387.1 mm, vias 0 -> 13
- net /D4: track 0.00 -> 383.5 mm, vias 0 -> 4
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Other:
- board size 223 x 137 mm -> 290 x 142.5 mm

Commit message: check designs for ALU (partial), SP, Shift register, register
Parts:
- added C1: 100n, Capacitor_THT:C_Disc_D5.0mm_W2.5mm_P5.00mm, F.Cu at (-53.1, 170.4)
- added C10: 100n, Capacitor_THT:C_Disc_D5.0mm_W2.5mm_P5.00mm, F.Cu at (-45.0, 178.5)
- added C11: 100n, Capacitor_THT:C_Disc_D5.0mm_W2.5mm_P5.00mm, F.Cu at (-45.0, 182.6)
- added C12: 100n, Capacitor_THT:C_Disc_D5.0mm_W2.5mm_P5.00mm, F.Cu at (-45.0, 186.6)
- added C13: 100n, Capacitor_THT:C_Disc_D5.0mm_W2.5mm_P5.00mm, F.Cu at (-45.0, 190.7)
- added C14: 100n, Capacitor_THT:C_Disc_D5.0mm_W2.5mm_P5.00mm, F.Cu at (-45.0, 194.7)
- added C15: 100n, Capacitor_THT:C_Disc_D5.0mm_W2.5mm_P5.00mm, F.Cu at (-36.8, 170.4)
- added C16: 220n, Capacitor_THT:C_Disc_D5.0mm_W2.5mm_P5.00mm, F.Cu at (-36.8, 174.4)
- added C17: 220n, Capacitor_THT:C_Disc_D5.0mm_W2.5mm_P5.00mm, F.Cu at (-36.8, 178.5)
- added C18: 220n, Capacitor_THT:C_Disc_D5.0mm_W2.5mm_P5.00mm, F.Cu at (-36.8, 182.6)
- added C19: 220n, Capacitor_THT:C_Disc_D5.0mm_W2.5mm_P5.00mm, F.Cu at (-36.8, 186.6)
- added C2: 100n, Capacitor_THT:C_Disc_D5.0mm_W2.5mm_P5.00mm, F.Cu at (-53.1, 174.4)
- added C20: 220n, Capacitor_THT:C_Disc_D5.0mm_W2.5mm_P5.00mm, F.Cu at (-36.8, 190.7)
- added C21: 47uF, Capacitor_THT:CP_Radial_D5.0mm_P2.50mm, F.Cu at (60.7, 231.1)
- added C22: 1uF, lncpu:CP_Radial_D4.0mm_P2.00mm-Large-Holes, F.Cu at (61.0, 238.5)
- added C3: 100n, Capacitor_THT:C_Disc_D5.0mm_W2.5mm_P5.00mm, F.Cu at (-53.1, 178.5)
- added C4: 100n, Capacitor_THT:C_Disc_D5.0mm_W2.5mm_P5.00mm, F.Cu at (-53.1, 182.6)
- added C5: 100n, Capacitor_THT:C_Disc_D5.0mm_W2.5mm_P5.00mm, F.Cu at (-53.1, 186.6)
- added C6: 100n, Capacitor_THT:C_Disc_D5.0mm_W2.5mm_P5.00mm, F.Cu at (-53.1, 190.7)
- added C7: 100n, Capacitor_THT:C_Disc_D5.0mm_W2.5mm_P5.00mm, F.Cu at (-53.1, 194.7)
- added C8: 100n, Capacitor_THT:C_Disc_D5.0mm_W2.5mm_P5.00mm, F.Cu at (-45.0, 170.4)
- added C9: 100n, Capacitor_THT:C_Disc_D5.0mm_W2.5mm_P5.00mm, F.Cu at (-45.0, 174.4)
- J2, J3: footprint Connector_PinSocket_2.54mm:PinSocket_1x08_P2.54mm_Vertical -> Connector_PinSocket_2.54mm:PinSocket_1x10_P2.54mm_Vertical
- U10, U11, U16, U17, U21: value 74HC86 -> 74LS86
- U12, U18, U5, U6, U9: value 74LS244 -> 74HCT541
- U13, U14: value 74AHC04 -> 74LS04
- U15, U2: value 74LS83 -> 74LS283
- U20: value LNCPU Type B Connector -> LNCPU Type B Header
- moved U12 236.5 mm to (129.5, 223.5), turned to 90 degrees
- moved U14 211.8 mm to (149.9, 255.3), turned to 90 degrees
- moved U19 203.2 mm to (57.1, 256.5), turned to 90 degrees
- moved U13 198.7 mm to (127.0, 241.3)
- moved U20 198.4 mm to (63.1, 220.7), turned to 180 degrees
- moved U1 167.7 mm to (172.7, 218.4), turned to 0 degrees
- moved J2 152.4 mm to (86.4, 236.2), turned to 0 degrees
- moved U9 147.7 mm to (219.5, 223.0), turned to 180 degrees
- moved U21 134.7 mm to (53.3, 167.0), turned to 0 degrees
- moved U10 134.6 mm to (236.2, 243.8), turned to -90 degrees
- moved U11 121.4 mm to (188.0, 251.5), turned to 90 degrees
- moved J3 103.7 mm to (238.8, 124.5), turned to 0 degrees
- moved U18 100.2 mm to (101.1, 179.0)
- moved U6 97.8 mm to (208.3, 177.8)
- moved U5 96.8 mm to (154.3, 176.5)
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Connections:
- J2 pad 1: /X0 -> GND
- J2 pad 2: /X1 -> /X0
- J2 pad 3: /X2 -> /X1
- J2 pad 4: /X3 -> /X2
- J2 pad 5: /X4 -> /X3
- J2 pad 6: /X5 -> /X4
- J2 pad 7: /X6 -> /X5
- J2 pad 8: /X7 -> /X6
- J3 pad 1: /Y0 -> GND
- J3 pad 2: /Y1 -> /Y0
- J3 pad 3: /Y2 -> /Y1
- J3 pad 4: /Y3 -> /Y2
- J3 pad 5: /Y4 -> /Y3
- J3 pad 6: /Y5 -> /Y4
- J3 pad 7: /Y6 -> /Y5
- J3 pad 8: /Y7 -> /Y6
- U10 pad 11: Net-(U9-I1a) -> Net-(U9-A1)
- U10 pad 3: Net-(U9-I3b) -> Net-(U9-A7)
- U10 pad 6: Net-(U9-I1b) -> Net-(U9-A5)
- U10 pad 8: Net-(U9-I3a) -> Net-(U9-A3)
- U11 pad 3: Net-(U9-I2b) -> Net-(U9-A6)
- U11 pad 6: Net-(U9-I0b) -> Net-(U9-A4)
- U11 pad 8: Net-(U9-I2a) -> Net-(U9-A2)
- U12 pad 11: Net-(U12-I0b) -> /D7
- U12 pad 12: /D3 -> /D6
- U12 pad 13: Net-(U12-I1b) -> /D5
- U12 pad 14: /D2 -> /D4
- U12 pad 15: Net-(U12-I2b) -> /D3
- U12 pad 16: /D1 -> /D2
- U12 pad 17: Net-(U12-I3b) -> /D1
- U12 pad 3: /D7 -> Net-(U12-A1)
- U12 pad 4: Net-(U12-I1a) -> Net-(U12-A2)
- U12 pad 5: /D6 -> Net-(U12-A3)
- U12 pad 6: Net-(U12-I2a) -> Net-(U12-A4)
- U12 pad 7: /D5 -> Net-(U12-A5)
- U12 pad 8: Net-(U12-I3a) -> Net-(U12-A6)
- U12 pad 9: /D4 -> Net-(U12-A7)
- U13 pad 10: Net-(U12-I3a) -> Net-(U12-A3)
- U13 pad 12: Net-(U12-I2a) -> Net-(U12-A2)
- U13 pad 2: Net-(U12-I3b) -> Net-(U12-A7)
- U13 pad 4: Net-(U12-I2b) -> Net-(U12-A6)
- U13 pad 6: Net-(U12-I1b) -> Net-(U12-A5)
- U13 pad 8: Net-(U12-I0b) -> Net-(U12-A4)
- U14 pad 2: Net-(U12-I1a) -> Net-(U12-A1)
- U15 pad 1: /X3 -> Net-(U15-S2)
- U15 pad 10: /X0 -> Net-(U15-S4)
- U15 pad 11: /Y_{xor}EN2_{0} -> /Y_{xor}EN2_{3}
- U15 pad 12: GND -> /X3
- U15 pad 13: Net-(U15-C0) -> Net-(U15-S3)
- U15 pad 14: Net-(U15-C4) -> /X2
- U15 pad 15: Net-(U15-S4) -> /Y_{xor}EN2_{2}
- U15 pad 16: /Y_{xor}EN2_{3} -> VCC
- U15 pad 2: Net-(U15-S3) -> /Y_{xor}EN2_{1}
- U15 pad 3: /X2 -> /X1
- U15 pad 4: /Y_{xor}EN2_{2} -> Net-(U15-S1)
- U15 pad 5: VCC -> /X0
- U15 pad 6: Net-(U15-S2) -> /Y_{xor}EN2_{0}
- U15 pad 7: /Y_{xor}EN2_{1} -> Net-(U15-C0)
- U15 pad 8: /X1 -> GND
- U15 pad 9: Net-(U15-S1) -> Net-(U15-C4)
- U18 pad 11: Net-(U18-I0b) -> /D7
- U18 pad 12: /D3 -> /D6
- U18 pad 13: Net-(U18-I1b) -> /D5
- U18 pad 14: /D2 -> /D4
- U18 pad 15: Net-(U18-I2b) -> /D3
- U18 pad 16: /D1 -> /D2
- U18 pad 17: Net-(U18-I3b) -> /D1
- U18 pad 3: /D7 -> Net-(U15-S2)
- U18 pad 4: Net-(U15-S2) -> Net-(U15-S3)
- U18 pad 5: /D6 -> Net-(U15-S4)
- U18 pad 6: Net-(U15-S3) -> Net-(U18-A4)
- U18 pad 7: /D5 -> Net-(U18-A5)
- U18 pad 8: Net-(U15-S4) -> Net-(U18-A6)
- U18 pad 9: /D4 -> Net-(U18-A7)
- U2 pad 1: /X7 -> Net-(U18-A5)
- U2 pad 10: /X4 -> Net-(U18-A7)
- U2 pad 11: /Y_{xor}EN2_{4} -> /Y_{xor}EN2_{7}
- U2 pad 12: GND -> /X7
- U2 pad 13: Net-(U15-C4) -> Net-(U18-A6)
- U2 pad 14: Net-(U2-C4) -> /X6
- U2 pad 15: Net-(U18-I3b) -> /Y_{xor}EN2_{6}
- U2 pad 16: /Y_{xor}EN2_{7} -> VCC
- U2 pad 2: Net-(U18-I2b) -> /Y_{xor}EN2_{5}
- U2 pad 3: /X6 -> /X5
- U2 pad 4: /Y_{xor}EN2_{6} -> Net-(U18-A4)
- U2 pad 5: VCC -> /X4
- U2 pad 6: Net-(U18-I1b) -> /Y_{xor}EN2_{4}
- U2 pad 7: /Y_{xor}EN2_{5} -> Net-(U15-C4)
- U2 pad 8: /X5 -> GND
- U2 pad 9: Net-(U18-I0b) -> Net-(U2-C4)
- U20 pad 10: /D3 -> Net-(U1-A1)
- U20 pad 11: Net-(U1-A0) -> /D4
- U20 pad 12: /D4 -> Net-(U1-A0)
- U20 pad 13: C_{out} -> /D5
- U20 pad 14: /D5 -> C_{out}
- U20 pad 15: unconnected-(U20-CTRL_{6}-Pad15) -> /D6
- U20 pad 16: /D6 -> unconnected-(U20-CTRL_{6}-Pad16)
- U20 pad 17: GND -> /D7
- U20 pad 18: /D7 -> GND
- U20 pad 20: GND -> unconnected-(U20-CLK2-Pad20)
- U20 pad 23: unconnected-(U20-CLK2-Pad23) -> GND
- U20 pad 3: Net-(U1-E1) -> /D0
- U20 pad 4: /D0 -> Net-(U1-E1)
- U20 pad 5: ~{ALU_{out}} -> /D1
- U20 pad 6: /D1 -> ~{ALU_{out}}
- U20 pad 7: Net-(U1-A2) -> /D2
- U20 pad 8: /D2 -> Net-(U1-A2)
- U20 pad 9: Net-(U1-A1) -> /D3
- U3 pad 11: Net-(U5-I1a) -> Net-(U5-A1)
- U3 pad 3: Net-(U5-I3b) -> Net-(U5-A7)
- U3 pad 6: Net-(U5-I1b) -> Net-(U5-A5)
- U3 pad 8: Net-(U5-I3a) -> Net-(U5-A3)
- U4 pad 3: Net-(U5-I2b) -> Net-(U5-A6)
- U4 pad 6: Net-(U5-I0b) -> Net-(U5-A4)
- U4 pad 8: Net-(U5-I2a) -> Net-(U5-A2)
- U5 pad 11: Net-(U5-I0b) -> /D7
- U5 pad 12: /D3 -> /D6
- U5 pad 13: Net-(U5-I1b) -> /D5
- U5 pad 14: /D2 -> /D4
- U5 pad 15: Net-(U5-I2b) -> /D3
- U5 pad 16: /D1 -> /D2
- U5 pad 17: Net-(U5-I3b) -> /D1
- U5 pad 3: /D7 -> Net-(U5-A1)
- U5 pad 4: Net-(U5-I1a) -> Net-(U5-A2)
- U5 pad 5: /D6 -> Net-(U5-A3)
- U5 pad 6: Net-(U5-I2a) -> Net-(U5-A4)
- U5 pad 7: /D5 -> Net-(U5-A5)
- U5 pad 8: Net-(U5-I3a) -> Net-(U5-A6)
- U5 pad 9: /D4 -> Net-(U5-A7)
- U6 pad 11: Net-(U6-I0b) -> /D7
- U6 pad 12: /D3 -> /D6
- U6 pad 13: Net-(U6-I1b) -> /D5
- U6 pad 14: /D2 -> /D4
- U6 pad 15: Net-(U6-I2b) -> /D3
- U6 pad 16: /D1 -> /D2
- U6 pad 17: Net-(U6-I3b) -> /D1
- U6 pad 3: /D7 -> Net-(U6-A1)
- U6 pad 4: Net-(U6-I1a) -> Net-(U6-A2)
- U6 pad 5: /D6 -> Net-(U6-A3)
- U6 pad 6: Net-(U6-I2a) -> Net-(U6-A4)
- U6 pad 7: /D5 -> Net-(U6-A5)
- U6 pad 8: Net-(U6-I3a) -> Net-(U6-A6)
- U6 pad 9: /D4 -> Net-(U6-A7)
- U7 pad 11: Net-(U6-I1a) -> Net-(U6-A1)
- U7 pad 3: Net-(U6-I3b) -> Net-(U6-A7)
- U7 pad 6: Net-(U6-I1b) -> Net-(U6-A5)
- U7 pad 8: Net-(U6-I3a) -> Net-(U6-A3)
- U8 pad 3: Net-(U6-I2b) -> Net-(U6-A6)
- U8 pad 6: Net-(U6-I0b) -> Net-(U6-A4)
- U8 pad 8: Net-(U6-I2a) -> Net-(U6-A2)
- U9 pad 11: Net-(U9-I0b) -> /D7
- U9 pad 12: /D3 -> /D6
- U9 pad 13: Net-(U9-I1b) -> /D5
- U9 pad 14: /D2 -> /D4
- U9 pad 15: Net-(U9-I2b) -> /D3
- U9 pad 16: /D1 -> /D2
- U9 pad 17: Net-(U9-I3b) -> /D1
- U9 pad 3: /D7 -> Net-(U9-A1)
- U9 pad 4: Net-(U9-I1a) -> Net-(U9-A2)
- U9 pad 5: /D6 -> Net-(U9-A3)
- U9 pad 6: Net-(U9-I2a) -> Net-(U9-A4)
- U9 pad 7: /D5 -> Net-(U9-A5)
- U9 pad 8: Net-(U9-I3a) -> Net-(U9-A6)
- U9 pad 9: /D4 -> Net-(U9-A7)
Routing:
- net GND: track 1154.4 -> 28.6 mm, vias 16 -> 0
- net VCC: track 916.3 -> 18.3 mm, vias 20 -> 0
- net Net-(U15-C0): track 453.7 -> 0.00 mm, vias 7 -> 0
- net Net-(U18-G1): track 436.6 -> 0.00 mm, vias 6 -> 0
- net /X4: track 430.0 -> 0.00 mm, vias 9 -> 0
- net /Y7: track 419.1 -> 0.00 mm, vias 6 -> 0
- net /X7: track 410.8 -> 0.00 mm, vias 4 -> 0
- net /X6: track 409.3 -> 0.00 mm, vias 9 -> 0
- net ~{ALU_{out}}: track 397.6 -> 0.00 mm, vias 6 -> 0
- net /X3: track 394.6 -> 0.00 mm, vias 4 -> 0
- net /X5: track 391.1 -> 0.00 mm, vias 8 -> 0
- net /X0: track 363.1 -> 0.00 mm, vias 7 -> 0
- net /Y5: track 351.6 -> 0.00 mm, vias 7 -> 0
- net /X1: track 347.5 -> 0.00 mm, vias 5 -> 0
- net /X2: track 345.9 -> 0.00 mm, vias 4 -> 0
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Other:
- board size 290 x 142.5 mm -> 200 x 150 mm
- board text added: "${REFERENCE}"

Commit message: readapt designs for BR, SP, SR, ALU
Parts:
- removed C1, C10, C11, C12, C13, C14, C15, C2, C3, C4, C5, C6, C7, C8, C9: 100n, Capacitor_THT:C_Disc_D5.0mm_W2.5mm_P5.00mm
- removed C16, C17, C18, C19, C20: 220n, Capacitor_THT:C_Disc_D5.0mm_W2.5mm_P5.00mm
- removed C21: 47uF, Capacitor_THT:CP_Radial_D5.0mm_P2.50mm
- removed C22: 1uF, lncpu:CP_Radial_D4.0mm_P2.00mm-Large-Holes
- removed J2: X_{in}, Connector_PinSocket_2.54mm:PinSocket_1x10_P2.54mm_Vertical
- removed J3: Y_{in}, Connector_PinSocket_2.54mm:PinSocket_1x10_P2.54mm_Vertical
- removed U1: 74LS138, Package_DIP:DIP-16_W7.62mm_LongPads
- removed U10, U11, U16, U17, U21: 74LS86, Package_DIP:DIP-14_W7.62mm_LongPads
- removed U12, U18, U5, U6, U9: 74HCT541, Package_DIP:DIP-20_W7.62mm_LongPads
- removed U13, U14: 74LS04, Package_DIP:DIP-14_W7.62mm_LongPads
- removed U15, U2: 74LS283, Package_DIP:DIP-16_W7.62mm_LongPads
- removed U19, U7, U8: 74LS08, Package_DIP:DIP-14_W7.62mm_LongPads
- removed U20: LNCPU Type B Header, lncpu:LNCPU_Type_B_Header
- removed U3, U4: 74LS32, Package_DIP:DIP-14_W7.62mm_LongPads
Routing:
- net /D4: track 118.9 -> 0.00 mm, vias 1 -> 0
- net /D3: track 118.8 -> 0.00 mm, vias 1 -> 0
- net /D5: track 117.4 -> 0.00 mm, vias 1 -> 0
- net /D2: track 117.3 -> 0.00 mm, vias 1 -> 0
- net /D1: track 117.2 -> 0.00 mm, vias 1 -> 0
- net /D0: track 117.1 -> 0.00 mm, vias 1 -> 0
- net /D6: track 116.6 -> 0.00 mm, vias 1 -> 0
- net /D7: track 115.9 -> 0.00 mm, vias 1 -> 0
- net GND: track 28.6 -> 0.00 mm
- net VCC: track 18.3 -> 0.00 mm
- net /Y0: track 1.40 -> 0.00 mm
Other:
- board text removed: "${REFERENCE}"
