File: v1/kicad/alu/alu/alu.kicad_sch (KiCad schematic)
At the start: 23 parts, among them J1 LNCPU_Type_A_connector,_male,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, J2 X_{in}, J3 Y_{in}, J4 ALU_C_flag_info_socket, U1 74LS138, U10 74HC86, U11 74HC86, U12 74LS244, U13 74AHC04, U14 74AHC04, U15 74LS83, U16 74HC86, U17 74HC86, U18 74LS244, U19 74LS08, U2 74LS83, U3 74LS32, U4 74LS32, U5 74LS244, U6 74LS244, U7 74LS08, U8 74LS08, U9 74LS244

Commit message: partial
Parts:
- removed J1: LNCPU_Type_A_connector,_male,_active_high_reset, LNCPU:LNCPU_TYPE_A_MALE, symbol lncpu:LNCPU_Type_A_connector,_male,_active_high_reset
- removed J4: ALU_C_flag_info_socket, Connector_PinSocket_2.54mm:PinSocket_1x02_P2.54mm_Vertical, symbol lncpu:ALU_C_flag_info_socket
- added unit 7 of U14
- added unit 1 of U19
- added U20: LNCPU Type B Connector, lncpu:LNCPU_Type_B_Header, symbol lncpu:LNCPU_Type_B_Connector
- added U21: 74HC86, Package_DIP:DIP-14_W7.62mm_LongPads, symbol 74xx:74HC86
- J2, J3: symbol lncpu:LNCPU DBUS socket -> lncpu:LNCPU_DBUS_Socket
- U1, U15, U2: footprint Package_DIP:DIP-16_W7.62mm -> Package_DIP:DIP-16_W7.62mm_LongPads
- U10, U11, U13, U14, U16, U17, U19, U3, U4, U7, U8: footprint Package_DIP:DIP-14_W7.62mm -> Package_DIP:DIP-14_W7.62mm_LongPads
- U12, U18, U5, U6, U9: footprint Package_DIP:DIP-20_W7.62mm -> Package_DIP:DIP-20_W7.62mm_LongPads
Connections:
- net D0: now also U20.4 (DBUS_{0})
- net D1: now also U20.6 (DBUS_{1})
- net D2: now also U20.8 (DBUS_{2})
- net D3: now also U20.10 (DBUS_{3})
- net D4: now also U20.12 (DBUS_{4})
- net D5: now also U20.14 (DBUS_{5})
- net D6: now also U20.16 (DBUS_{6})
- net D7: now also U20.18 (DBUS_{7})
- net GND: now also U14.13, U14.7 (GND), U20.1 (GND), U20.17 (GND), U20.20 (GND), U20.22 (GND), U21.10, U21.12, U21.13, U21.4, U21.5, U21.7 (GND), U21.9; no longer U14.13, U14.7 (GND), U19.1, U19.2
- net VCC: now also U14.14 (VCC), U20.2 (VCC), U20.24 (VCC), U21.14 (VCC); no longer U14.14 (VCC)
- net ~{ALU_{out}}: now also U20.5 (CTRL_{1})
- net ~{EN2}: no longer U14.9
- net at U14.6, U15.13 (C0), U16.1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: now also U21.1
- net at U18.1 (OEa), U19.6: now also U14.9
- net at U14.8: now also U19.2
- net at U1.1 (A0): now also U20.11 (CTRL_{4})
- net at U1.2 (A1): now also U20.9 (CTRL_{3})
- net at U1.3 (A2): now also U20.7 (CTRL_{2})
- net at U1.4 (E1): now also U20.3 (CTRL_{0})
- net at U2.14 (C4): now also U21.2
- new net: U19.1, U21.3
- new net C_{out}: U19.3, U20.13 (CTRL_{5})
- no-connect marks 11 -> 13
Other:
- moved on the sheet: J2, J3, U19D

Commit message: check designs for ALU (partial), SP, Shift register, register
Parts:
- added C1, C10, C11, C12, C13, C14, C15, C2, C3, C4, C5, C6, C7, C8, C9: 100n, Capacitor_THT:C_Disc_D5.0mm_W2.5mm_P5.00mm, symbol Device:C
- added C16, C17, C18, C19, C20: 220n, Capacitor_THT:C_Disc_D5.0mm_W2.5mm_P5.00mm, symbol Device:C
- added C21: 47uF, Capacitor_THT:CP_Radial_D5.0mm_P2.50mm, symbol Device:C_Polarized
- added C22: 1uF, lncpu:CP_Radial_D4.0mm_P2.00mm-Large-Holes, symbol Device:C_Polarized
- added unit 3 of U21
- added unit 1 of U21
- added unit 5 of U21
- added unit 4 of U21
- J2, J3: footprint Connector_PinSocket_2.54mm:PinSocket_1x08_P2.54mm_Vertical -> Connector_PinSocket_2.54mm:PinSocket_1x10_P2.54mm_Vertical; symbol lncpu:LNCPU_DBUS_Socket -> lncpu:LNCPU_8B_Socket
- U10, U11, U16, U17, U21: value 74HC86 -> 74LS86; symbol 74xx:74HC86 -> 74xx:74LS86
- U12, U18, U5, U6, U9: value 74LS244 -> 74HCT541; symbol 74xx:74LS244 -> 74xx:74HCT541
- U13, U14: value 74AHC04 -> 74LS04; symbol 74xx:74AHC04 -> 74xx:74LS04
- U15, U2: value 74LS83 -> 74LS283; symbol 74xx:74LS83 -> 74xx:74LS283
- U20: value LNCPU Type B Connector -> LNCPU Type B Header; symbol lncpu:LNCPU_Type_B_Connector -> lncpu:LNCPU_Type_B_Header
Connections:
- net C_{out}: now also U20.14 (CTRL_{5}); no longer U20.13 (CTRL_{5})
- net D0: now also U20.3 (DBUS_{0}); no longer U20.4 (DBUS_{0})
- net D1: now also U12.17 (Y1), U18.17 (Y1), U20.5 (DBUS_{1}), U5.17 (Y1), U6.17 (Y1), U9.17 (Y1); no longer U12.16 (O1a), U18.16 (O1a), U20.6 (DBUS_{1}), U5.16 (O1a), U6.16 (O1a), U9.16 (O1a)
- net D2: now also U12.16 (Y2), U18.16 (Y2), U20.7 (DBUS_{2}), U5.16 (Y2), U6.16 (Y2), U9.16 (Y2); no longer U12.14 (O2a), U18.14 (O2a), U20.8 (DBUS_{2}), U5.14 (O2a), U6.14 (O2a), U9.14 (O2a)
- net D3: now also U12.15 (Y3), U18.15 (Y3), U20.9 (DBUS_{3}), U5.15 (Y3), U6.15 (Y3), U9.15 (Y3); no longer U12.12 (O3a), U18.12 (O3a), U20.10 (DBUS_{3}), U5.12 (O3a), U6.12 (O3a), U9.12 (O3a)
- net D4: now also U12.14 (Y4), U18.14 (Y4), U20.11 (DBUS_{4}), U5.14 (Y4), U6.14 (Y4), U9.14 (Y4); no longer U12.9 (O0b), U18.9 (O0b), U20.12 (DBUS_{4}), U5.9 (O0b), U6.9 (O0b), U9.9 (O0b)
- net D5: now also U12.13 (Y5), U18.13 (Y5), U20.13 (DBUS_{5}), U5.13 (Y5), U6.13 (Y5), U9.13 (Y5); no longer U12.7 (O1b), U18.7 (O1b), U20.14 (DBUS_{5}), U5.7 (O1b), U6.7 (O1b), U9.7 (O1b)
- net D6: now also U12.12 (Y6), U18.12 (Y6), U20.15 (DBUS_{6}), U5.12 (Y6), U6.12 (Y6), U9.12 (Y6); no longer U12.5 (O2b), U18.5 (O2b), U20.16 (DBUS_{6}), U5.5 (O2b), U6.5 (O2b), U9.5 (O2b)
- net D7: now also U12.11 (Y7), U18.11 (Y7), U20.17 (DBUS_{7}), U5.11 (Y7), U6.11 (Y7), U9.11 (Y7); no longer U12.3 (O3b), U18.3 (O3b), U20.18 (DBUS_{7}), U5.3 (O3b), U6.3 (O3b), U9.3 (O3b)
- net GND: now also J2.1 (GND), J2.10 (GND), J3.1 (GND), J3.10 (GND), U15.8 (GND), U2.8 (GND), U20.18 (GND), U20.23 (GND), C1.2, C10.1, C11.1, C12.1, C13.1, C14.2, C15.2, C16.2, C17.2, C18.2, C19.2, C2.1, C20.2, C21.2, C22.2, C3.1, C4.1, C5.1, C6.1, C7.1, C8.1, C9.1, U21.10, U21.12, U21.13, U21.7 (GND), U21.9; no longer U15.12 (GND), U2.12 (GND), U20.17 (GND), U20.20 (GND), U21.10, U21.12, U21.13, U21.7 (GND), U21.9
- net VCC: now also U15.16 (VCC), U2.16 (VCC), C1.1, C10.2, C11.2, C12.2, C13.2, C14.1, C15.1, C16.1, C17.1, C18.1, C19.1, C2.2, C20.1, C21.1, C22.1, C3.2, C4.2, C5.2, C6.2, C7.2, C8.2, C9.2, U21.14 (VCC); no longer U15.5 (VCC), U2.5 (VCC), U21.14 (VCC)
- net X0: now also J2.2 (D0), U15.5 (A1); no longer J2.1 (D0), U15.10 (A1)
- net X1: now also J2.3 (D1), U15.3 (A2); no longer J2.2 (D1), U15.8 (A2)
- net X2: now also J2.4 (D2), U15.14 (A3); no longer J2.3 (D2), U15.3 (A3)
- net X3: now also J2.5 (D3), U15.12 (A4); no longer J2.4 (D3), U15.1 (A4)
- net X4: now also J2.6 (D4), U2.5 (A1); no longer J2.5 (D4), U2.10 (A1)
- net X5: now also J2.7 (D5), U2.3 (A2); no longer J2.6 (D5), U2.8 (A2)
- net X6: now also J2.8 (D6), U2.14 (A3); no longer J2.7 (D6), U2.3 (A3)
- net X7: now also J2.9 (D7), U2.12 (A4); no longer J2.8 (D7), U2.1 (A4)
- net Y0: now also J3.2 (D0); no longer J3.1 (D0)
- net Y1: now also J3.3 (D1); no longer J3.2 (D1)
- net Y2: now also J3.4 (D2); no longer J3.3 (D2)
- net Y3: now also J3.5 (D3); no longer J3.4 (D3)
- net Y4: now also J3.6 (D4); no longer J3.5 (D4)
- net Y5: now also J3.7 (D5); no longer J3.6 (D5)
- net Y6: now also J3.8 (D6); no longer J3.7 (D6)
- net Y7: now also J3.9 (D7); no longer J3.8 (D7)
- net Y_{xor}EN2_{0}: now also U15.6 (B1); no longer U15.11 (B1)
- net Y_{xor}EN2_{1}: now also U15.2 (B2); no longer U15.7 (B2)
- net Y_{xor}EN2_{2}: now also U15.15 (B3); no longer U15.4 (B3)
- net Y_{xor}EN2_{3}: now also U15.11 (B4); no longer U15.16 (B4)
- net Y_{xor}EN2_{4}: now also U2.6 (B1); no longer U2.11 (B1)
- net Y_{xor}EN2_{5}: now also U2.2 (B2); no longer U2.7 (B2)
- net Y_{xor}EN2_{6}: now also U2.15 (B3); no longer U2.4 (B3)
- net Y_{xor}EN2_{7}: now also U2.11 (B4); no longer U2.16 (B4)
- net ~{ALU_{out}}: now also U20.6 (CTRL_{1}); no longer U20.5 (CTRL_{1})
- net at U14.6, U16.1, U16.12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: now also U15.7 (C0), U21.1; no longer U15.13 (C0), U21.1
- net at U2.13 (S3): now also U18.8 (A6); no longer U15.14 (C4)
- net at U18.6 (A4): now also U2.4 (S1); no longer U15.2 (S3)
- net at U18.4 (A2): now also U15.13 (S3); no longer U15.6 (S2)
- net at U18.2 (A0): now also U15.4 (S1); no longer U15.9 (S1)
- net at U2.9 (C4): now also U21.2; no longer U18.11 (I0b)
- net at U11.6: now also U9.6 (A4); no longer U9.11 (I0b)
- net at U13.12: now also U12.4 (A2); no longer U12.6 (I2a)
- net at U7.11: now also U6.3 (A1); no longer U6.4 (I1a)
- net at U3.6: now also U5.7 (A5); no longer U5.13 (I1b)
- net at U11.3: now also U9.8 (A6); no longer U9.15 (I2b)
- net at U13.6: now also U12.7 (A5); no longer U12.13 (I1b)
- net at U4.6: now also U5.6 (A4); no longer U5.11 (I0b)
- net at U19.1: now also U21.3; no longer U21.3
- net at U8.6: now also U6.6 (A4); no longer U6.11 (I0b)
- net at U10.6: now also U9.7 (A5); no longer U9.13 (I1b)
- net at U10.3: now also U9.9 (A7); no longer U9.17 (I3b)
- net at U10.11: now also U9.3 (A1); no longer U9.4 (I1a)
- net at U11.8: now also U9.4 (A2); no longer U9.6 (I2a)
- net at U10.8: now also U9.5 (A3); no longer U9.8 (I3a)
- net at U8.8: now also U6.4 (A2); no longer U6.6 (I2a)
- net at U1.1 (A0): now also U20.12 (CTRL_{4}); no longer U20.11 (CTRL_{4})
- net at U1.2 (A1): now also U20.10 (CTRL_{3}); no longer U20.9 (CTRL_{3})
- net at U1.3 (A2): now also U20.8 (CTRL_{2}); no longer U20.7 (CTRL_{2})
- net at U1.4 (E1): now also U20.4 (CTRL_{0}); no longer U20.3 (CTRL_{0})
- net at U4.3: now also U5.8 (A6); no longer U5.15 (I2b)
- net at U3.3: now also U5.9 (A7); no longer U5.17 (I3b)
- net at U3.11: now also U5.3 (A1); no longer U5.4 (I1a)
- net at U4.8: now also U5.4 (A2); no longer U5.6 (I2a)
- net at U3.8: now also U5.5 (A3); no longer U5.8 (I3a)
- net at U13.2: now also U12.9 (A7); no longer U12.17 (I3b)
- net at U7.6: now also U6.7 (A5); no longer U6.13 (I1b)
- net at U13.8: now also U12.6 (A4); no longer U12.11 (I0b)
- net at U13.4: now also U12.8 (A6); no longer U12.15 (I2b)
- net at U14.2: now also U12.3 (A1); no longer U12.4 (I1a)
- net at U13.10: now also U12.5 (A3); no longer U12.8 (I3a)
- net at U7.3: now also U6.9 (A7); no longer U6.17 (I3b)
- net at U7.8: now also U6.5 (A3); no longer U6.8 (I3a)
- net at U8.3: now also U6.8 (A6); no longer U6.15 (I2b)
- new net: U15.1 (S2), U18.3 (A1)
- new net: U15.10 (S4), U18.5 (A3)
- new net: U15.9 (C4), U2.7 (C0)
- new net: U18.7 (A5), U2.1 (S2)
- new net: U18.9 (A7), U2.10 (S4)
Other:
- moved on the sheet: U20

Commit message: readapt designs for BR, SP, SR, ALU
Connections:
- net X0: now also U10.2, U14.1, U3.2, U7.2; no longer U11.13, U14.3, U4.13, U8.13
- net X1: now also U10.5, U14.3, U3.5, U7.5; no longer U10.13, U14.1, U3.13, U7.13
- net X2: now also U10.10, U13.1, U3.10, U7.10; no longer U11.10, U13.13, U4.10, U8.10
- net X3: now also U10.13, U13.3, U3.13, U7.13; no longer U10.10, U13.11, U3.10, U7.10
- net X4: now also U11.2, U13.5, U4.2, U8.2; no longer U11.5, U13.9, U4.5, U8.5
- net X5: now also U11.5, U13.9, U4.5, U8.5; no longer U10.5, U13.5, U3.5, U7.5
- net X6: now also U11.10, U13.11, U4.10, U8.10; no longer U11.2, U13.3, U4.2, U8.2
- net X7: now also U11.13, U13.13, U4.13, U8.13; no longer U10.2, U13.1, U3.2, U7.2
- net Y0: now also U10.1, U16.2, U3.1, U7.1; no longer U11.12, U17.13, U4.12, U8.12
- net Y1: now also U10.4, U16.5, U3.4, U7.4; no longer U10.12, U16.13, U3.12, U7.12
- net Y2: now also U10.9, U16.10, U3.9, U7.9; no longer U11.9, U17.10, U4.9, U8.9
- net Y3: now also U10.12, U16.13, U3.12, U7.12; no longer U10.9, U16.10, U3.9, U7.9
- net Y4: now also U11.1, U17.2, U4.1, U8.1; no longer U11.4, U17.5, U4.4, U8.4
- net Y5: now also U11.4, U17.5, U4.4, U8.4; no longer U10.4, U16.5, U3.4, U7.4
- net Y6: now also U11.9, U17.10, U4.9, U8.9; no longer U11.1, U17.2, U4.1, U8.1
- net Y7: now also U11.12, U17.13, U4.12, U8.12; no longer U10.1, U16.2, U3.1, U7.1
- net Y_{xor}EN2_{0}: now also U16.3; no longer U17.11
- net Y_{xor}EN2_{1}: now also U16.6; no longer U16.11
- net Y_{xor}EN2_{2}: now also U16.8; no longer U17.8
- net Y_{xor}EN2_{3}: now also U16.11; no longer U16.8
- net Y_{xor}EN2_{4}: now also U17.3; no longer U17.6
- net Y_{xor}EN2_{5}: now also U17.6; no longer U16.6
- net Y_{xor}EN2_{6}: now also U17.8; no longer U17.3
- net Y_{xor}EN2_{7}: now also U17.11; no longer U16.3
- net at U9.2 (A0): now also U10.3; no longer U11.11
- net at U9.6 (A4): now also U11.3; no longer U11.6
- net at U13.12: now also U12.9 (A7); no longer U12.4 (A2)
- net at U6.3 (A1): now also U7.6; no longer U7.11
- net at U3.6: now also U5.3 (A1); no longer U5.7 (A5)
- net at U9.8 (A6): now also U11.8; no longer U11.3
- net at U13.6: now also U12.6 (A4); no longer U12.7 (A5)
- net at U5.6 (A4): now also U4.3; no longer U4.6
- net at U6.6 (A4): now also U8.3; no longer U8.6
- net at U10.11: now also U9.5 (A3); no longer U9.3 (A1)
- net at U9.4 (A2): now also U10.8; no longer U11.8
- net at U10.6: now also U9.3 (A1); no longer U9.7 (A5)
- net at U9.9 (A7): now also U11.11; no longer U10.3
- net at U14.4: now also U12.3 (A1); no longer U12.2 (A0)
- net at U6.4 (A2): now also U7.8; no longer U8.8
- net at U5.8 (A6): now also U4.8; no longer U4.3
- net at U5.2 (A0): now also U3.3; no longer U4.11
- net at U3.11: now also U5.5 (A3); no longer U5.3 (A1)
- net at U5.4 (A2): now also U3.8; no longer U4.8
- net at U5.9 (A7): now also U4.11; no longer U3.3
- net at U13.2: now also U12.4 (A2); no longer U12.9 (A7)
- net at U6.7 (A5): now also U8.6; no longer U7.6
- net at U6.2 (A0): now also U7.3; no longer U8.11
- net at U13.8: now also U12.7 (A5); no longer U12.6 (A4)
- net at U13.4: now also U12.5 (A3); no longer U12.8 (A6)
- net at U14.2: now also U12.2 (A0); no longer U12.3 (A1)
- net at U13.10: now also U12.8 (A6); no longer U12.5 (A3)
- net at U6.9 (A7): now also U8.11; no longer U7.3
- net at U6.5 (A3): now also U7.11; no longer U7.8
- net at U6.8 (A6): now also U8.8; no longer U8.3
- new net: U11.6, U9.7 (A5)
- new net: U4.6, U5.7 (A5)
