File: v1/kicad/alu/alu_operand_selector/alu_operand_selector.kicad_sch (KiCad schematic)
At the start: 19 parts, among them J1 LNCPU ALU Operand Selector so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, J10 OP_{out}, J2 A_{in}, J3 B_{in}, J4 C_{in}, J5 D_{in}, J6 E_{in}, J7 F_{in}, J8 G_{in}, J9 H_{in}, U1 74HC138, U2 74LS244, U3 74HC244, U4 74HC244, U5 74HC244, U6 74HC244, U7 74HC244, U8 74HC244, U9 74HC244

Commit message: Add alu from old design
Parts:
- removed J1: LNCPU ALU Operand Selector socket, male, Connector_PinHeader_2.54mm:PinHeader_1x08_P2.54mm_Horizontal, symbol lncpu:LNCPU ALU Operand Selector socket, male
- added U10: LNCPU Type C Connector, symbol lncpu:LNCPU_Type_C_Connector
- J10, J2, J3, J4, J5, J6, J7, J8, J9: symbol lncpu:LNCPU_DBUS_SOCKET -> lncpu:LNCPU_DBUS_Socket
Connections:
- net at U1.16 (VCC), U2.20 (VCC), U3.20 (VCC)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: now also U10.16 (VCC), U10.2 (VCC)
- net at U1.3 (A2): now also U10.4 (CTRL_{1})
- net at U1.2 (A1): now also U10.5 (CTRL_{2})
- net at U1.1 (A0): now also U10.6 (CTRL_{3})
- net at U1.6 (E3): now also U10.3 (CTRL_{0})
- net at U1.4 (~{E1}), U1.5 (~{E2}), U1.8 (GND)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: now also U10.1 (GND), U10.10 (GND), U10.12 (GND), U10.14 (GND)
- no-connect marks 0 -> 6
Other:
- moved on the sheet: J10, J2, J3, J4, J5, J6, J7, J8, J9

Commit message: partial
Parts:
- U1: footprint Package_DIP:DIP-16_W7.62mm -> Package_DIP:DIP-16_W7.62mm_LongPads
- U10: footprint (none) -> lncpu:LNCPU_Type_C_Header
- U2, U3, U4, U5, U6, U7, U8, U9: footprint Package_DIP:DIP-20_W7.62mm -> Package_DIP:DIP-20_W7.62mm_LongPads
Changed lines of the file:
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@@
 			)
 		)
-		(property "Footprint" "Package_DIP:DIP-20_W7.62mm"
+		(property "Footprint" "Package_DIP:DIP-20_W7.62mm_LongPads"
 			(at 163.83 168.91 0)
 			(effects
@@
 			)
 		)
-		(property "Footprint" "Package_DIP:DIP-20_W7.62mm"
+		(property "Footprint" "Package_DIP:DIP-20_W7.62mm_LongPads"
 			(at 163.83 452.12 0)
 			(effects
@@
 			)
 		)
-		(property "Footprint" ""
+		(property "Footprint" "lncpu:LNCPU_Type_C_Header"
 			(at 109.22 95.25 0)
 			(effects
@@
 			)
 		)
-		(property "Footprint" "Package_DIP:DIP-20_W7.62mm"
+		(property "Footprint" "Package_DIP:DIP-20_W7.62mm_LongPads"
 			(at 163.83 123.19 0)
 			(effects
@@
 			)
 		)
-		(property "Footprint" "Package_DIP:DIP-20_W7.62mm"
+		(property "Footprint" "Package_DIP:DIP-20_W7.62mm_LongPads"
 			(at 163.83 312.42 0)
 			(effects
@@
 			)
 		)
-		(property "Footprint" "Package_DIP:DIP-16_W7.62mm"
+		(property "Footprint" "Package_DIP:DIP-16_W7.62mm_LongPads"
 			(at 163.83 80.01 0)
 			(effects
@@
 			)
 		)
-		(property "Footprint" "Package_DIP:DIP-20_W7.62mm"
+		(property "Footprint" "Package_DIP:DIP-20_W7.62mm_LongPads"
 			(at 163.83 405.13 0)
 			(effects
@@
 			)
 		)
-		(property "Footprint" "Package_DIP:DIP-20_W7.62mm"
+		(property "Footprint" "Package_DIP:DIP-20_W7.62mm_LongPads"
 			(at 163.83 215.9 0)
 			(effects
@@
 			)
 		)
-		(property "Footprint" "Package_DIP:DIP-20_W7.62mm"
+		(property "Footprint" "Package_DIP:DIP-20_W7.62mm_LongPads"
 			(at 163.83 358.14 0)
 			(effects
@@
 			)
 		)
-		(property "Footprint" "Package_DIP:DIP-20_W7.62mm"
+		(property "Footprint" "Package_DIP:DIP-20_W7.62mm_LongPads"
 			(at 163.83 262.89 0)
 			(effects

Commit message: readapt designs for BR, SP, SR, ALU
Parts:
- removed J10: OP_{out}, Connector_PinSocket_2.54mm:PinSocket_1x08_P2.54mm_Vertical, symbol lncpu:LNCPU_DBUS_Socket
- added C1: 47u, Capacitor_THT:CP_Radial_D5.0mm_P2.00mm, symbol Device:C_Polarized
- added C10, C11, C4, C5, C6, C7, C8, C9: 220n, Capacitor_THT:C_Disc_D5.0mm_W2.5mm_P2.50mm, symbol Device:C
- added C2: 1u, lncpu:CP_Radial_D4.0mm_P2.00mm-Large-Holes, symbol Device:C_Polarized
- added C3: 100n, Capacitor_THT:C_Disc_D5.0mm_W2.5mm_P2.50mm, symbol Device:C
- J1: renamed from J2; footprint Connector_PinSocket_2.54mm:PinSocket_1x08_P2.54mm_Vertical -> Connector_PinSocket_2.54mm:PinSocket_1x10_P2.54mm_Vertical; symbol lncpu:LNCPU_DBUS_Socket -> lncpu:LNCPU_8B_Socket
- J2: renamed from J3; footprint Connector_PinSocket_2.54mm:PinSocket_1x08_P2.54mm_Vertical -> Connector_PinSocket_2.54mm:PinSocket_1x10_P2.54mm_Vertical; symbol lncpu:LNCPU_DBUS_Socket -> lncpu:LNCPU_8B_Socket
- J3: renamed from J4; footprint Connector_PinSocket_2.54mm:PinSocket_1x08_P2.54mm_Vertical -> Connector_PinSocket_2.54mm:PinSocket_1x10_P2.54mm_Vertical; symbol lncpu:LNCPU_DBUS_Socket -> lncpu:LNCPU_8B_Socket
- J4: renamed from J5; footprint Connector_PinSocket_2.54mm:PinSocket_1x08_P2.54mm_Vertical -> Connector_PinSocket_2.54mm:PinSocket_1x10_P2.54mm_Vertical; symbol lncpu:LNCPU_DBUS_Socket -> lncpu:LNCPU_8B_Socket
- J5: renamed from J6; footprint Connector_PinSocket_2.54mm:PinSocket_1x08_P2.54mm_Vertical -> Connector_PinSocket_2.54mm:PinSocket_1x10_P2.54mm_Vertical; symbol lncpu:LNCPU_DBUS_Socket -> lncpu:LNCPU_8B_Socket
- J6: renamed from J7; footprint Connector_PinSocket_2.54mm:PinSocket_1x08_P2.54mm_Vertical -> Connector_PinSocket_2.54mm:PinSocket_1x10_P2.54mm_Vertical; symbol lncpu:LNCPU_DBUS_Socket -> lncpu:LNCPU_8B_Socket
- J7: renamed from J8; footprint Connector_PinSocket_2.54mm:PinSocket_1x08_P2.54mm_Vertical -> Connector_PinSocket_2.54mm:PinSocket_1x10_P2.54mm_Vertical; symbol lncpu:LNCPU_DBUS_Socket -> lncpu:LNCPU_8B_Socket
- J8: renamed from J9; footprint Connector_PinSocket_2.54mm:PinSocket_1x08_P2.54mm_Vertical -> Connector_PinSocket_2.54mm:PinSocket_1x10_P2.54mm_Vertical; symbol lncpu:LNCPU_DBUS_Socket -> lncpu:LNCPU_8B_Socket
- U1: renamed from U10; value LNCPU Type C Connector -> LNCPU Type B Header; footprint lncpu:LNCPU_Type_C_Header -> lncpu:LNCPU_Type_B_Header; symbol lncpu:LNCPU_Type_C_Connector -> lncpu:LNCPU_Type_B_Header
- U10: renamed from U9; value 74HC244 -> 74HCT541; symbol 74xx:74LS244 -> 74xx:74HCT541
- U3: renamed from U2; value 74LS244 -> 74HCT541; symbol 74xx:74LS244 -> 74xx:74HCT541
- U4: renamed from U3; value 74HC244 -> 74HCT541; symbol 74xx:74LS244 -> 74xx:74HCT541
- U5: renamed from U4; value 74HC244 -> 74HCT541; symbol 74xx:74LS244 -> 74xx:74HCT541
- U6: renamed from U5; value 74HC244 -> 74HCT541; symbol 74xx:74LS244 -> 74xx:74HCT541
- U7: renamed from U6; value 74HC244 -> 74HCT541; symbol 74xx:74LS244 -> 74xx:74HCT541
- U8: renamed from U7; value 74HC244 -> 74HCT541; symbol 74xx:74LS244 -> 74xx:74HCT541
- U9: renamed from U8; value 74HC244 -> 74HCT541; symbol 74xx:74LS244 -> 74xx:74HCT541
- renumbered U1 to U2
Connections:
- net EN.A: no longer U3.19 (OEb)
- net EN.B: no longer U4.19 (OEb)
- net EN.C: no longer U5.19 (OEb)
- net EN.D: no longer U6.19 (OEb)
- net EN.E: no longer U7.19 (OEb)
- net EN.F: no longer U8.19 (OEb)
- net EN.G: no longer U9.19 (OEb)
- net EN.H: no longer U10.19 (OEb)
- net OP_{out}0: now also U1.17 (DBUS_{7})
- net OP_{out}1: now also U1.15 (DBUS_{6}), U10.17 (Y1), U3.17 (Y1), U4.17 (Y1), U5.17 (Y1), U6.17 (Y1), U7.17 (Y1), U8.17 (Y1), U9.17 (Y1); no longer U10.16 (O1a), U3.16 (O1a), U4.16 (O1a), U5.16 (O1a), U6.16 (O1a), U7.16 (O1a), U8.16 (O1a), U9.16 (O1a)
- net OP_{out}2: now also U1.13 (DBUS_{5}), U10.16 (Y2), U3.16 (Y2), U4.16 (Y2), U5.16 (Y2), U6.16 (Y2), U7.16 (Y2), U8.16 (Y2), U9.16 (Y2); no longer U10.14 (O2a), U3.14 (O2a), U4.14 (O2a), U5.14 (O2a), U6.14 (O2a), U7.14 (O2a), U8.14 (O2a), U9.14 (O2a)
- net OP_{out}3: now also U1.11 (DBUS_{4}), U10.15 (Y3), U3.15 (Y3), U4.15 (Y3), U5.15 (Y3), U6.15 (Y3), U7.15 (Y3), U8.15 (Y3), U9.15 (Y3); no longer U10.12 (O3a), U3.12 (O3a), U4.12 (O3a), U5.12 (O3a), U6.12 (O3a), U7.12 (O3a), U8.12 (O3a), U9.12 (O3a)
- net OP_{out}4: now also U1.9 (DBUS_{3}), U10.14 (Y4), U3.14 (Y4), U4.14 (Y4), U5.14 (Y4), U6.14 (Y4), U7.14 (Y4), U8.14 (Y4), U9.14 (Y4); no longer U10.9 (O0b), U3.9 (O0b), U4.9 (O0b), U5.9 (O0b), U6.9 (O0b), U7.9 (O0b), U8.9 (O0b), U9.9 (O0b)
- net OP_{out}5: now also U1.7 (DBUS_{2}), U10.13 (Y5), U3.13 (Y5), U4.13 (Y5), U5.13 (Y5), U6.13 (Y5), U7.13 (Y5), U8.13 (Y5), U9.13 (Y5); no longer U10.7 (O1b), U3.7 (O1b), U4.7 (O1b), U5.7 (O1b), U6.7 (O1b), U7.7 (O1b), U8.7 (O1b), U9.7 (O1b)
- net OP_{out}6: now also U1.5 (DBUS_{1}), U10.12 (Y6), U3.12 (Y6), U4.12 (Y6), U5.12 (Y6), U6.12 (Y6), U7.12 (Y6), U8.12 (Y6), U9.12 (Y6); no longer U10.5 (O2b), U3.5 (O2b), U4.5 (O2b), U5.5 (O2b), U6.5 (O2b), U7.5 (O2b), U8.5 (O2b), U9.5 (O2b)
- net OP_{out}7: now also U1.3 (DBUS_{0}), U10.11 (Y7), U3.11 (Y7), U4.11 (Y7), U5.11 (Y7), U6.11 (Y7), U7.11 (Y7), U8.11 (Y7), U9.11 (Y7); no longer U10.3 (O3b), U3.3 (O3b), U4.3 (O3b), U5.3 (O3b), U6.3 (O3b), U7.3 (O3b), U8.3 (O3b), U9.3 (O3b)
- net at J6.1 (GND): now also J1.1 (GND), J2.1 (GND), J3.1 (GND), J4.1 (GND), J5.1 (GND), J7.1 (GND), J8.1 (GND), U1.1 (GND), U1.18 (GND), U1.22 (GND), U1.23 (GND), U10.10 (GND), U2.8 (GND), U3.10 (GND), U4.10 (GND), U5.10 (GND), U6.10 (GND), U7.10 (GND), U8.10 (GND), U9.10 (GND), C1.2, C10.2, C11.2, C2.2, C3.2, C4.2, C5.2, C6.2, C7.2, C8.2, C9.2; no longer U8.17 (I3b)
- net at J6.2 (D0): now also U8.2 (A0); no longer U8.15 (I2b)
- net at J6.3 (D1): now also U8.3 (A1); no longer U8.13 (I1b)
- net at J6.4 (D2): now also U8.4 (A2); no longer U8.11 (I0b)
- net at J6.5 (D3): now also U8.5 (A3); no longer U8.8 (I3a)
- net at J6.7 (D5): now also U8.7 (A5); no longer U8.4 (I1a)
- net at J6.8 (D6): now also U8.8 (A6); no longer U8.2 (I0a)
- net at J2.4 (D2): now also U4.4 (A2); no longer U4.11 (I0b)
- net at J2.3 (D1): now also U4.3 (A1); no longer U4.13 (I1b)
- net at J2.2 (D0): now also U4.2 (A0); no longer U4.15 (I2b)
- net at J2.8 (D6): now also U4.8 (A6); no longer U4.2 (I0a)
- net at U1.2 (VCC), U10.20 (VCC), U2.16 (VCC)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: now also J1.10 (VCC), J2.10 (VCC), J3.10 (VCC), J4.10 (VCC), J5.10 (VCC), J6.10 (VCC), J7.10 (VCC), J8.10 (VCC), U1.24 (VCC), U2.6 (E3), C1.1, C10.1, C11.1, C2.1, C3.1, C4.1, C5.1, C6.1, C7.1, C8.1, C9.1; no longer U1.16 (VCC)
- net at J2.7 (D5): now also U4.7 (A5); no longer U4.4 (I1a)
- net at J2.5 (D3): now also U4.5 (A3); no longer U4.8 (I3a)
- net at J8.4 (D2): now also U10.4 (A2); no longer U10.11 (I0b)
- net at J8.3 (D1): now also U10.3 (A1); no longer U10.13 (I1b)
- net at J8.2 (D0): now also U10.2 (A0); no longer U10.15 (I2b)
- net at J8.8 (D6): now also U10.8 (A6); no longer U10.2 (I0a)
- net at J8.7 (D5): now also U10.7 (A5); no longer U10.4 (I1a)
- net at J8.5 (D3): now also U10.5 (A3); no longer U10.8 (I3a)
- net at U2.3 (A2): now also U1.10 (CTRL_{3}); no longer U1.4 (CTRL_{1})
- net at U2.2 (A1): now also U1.8 (CTRL_{2}); no longer U1.5 (CTRL_{2})
- net at J1.4 (D2): now also U3.4 (A2); no longer U3.11 (I0b)
- net at J1.3 (D1): now also U3.3 (A1); no longer U3.13 (I1b)
- net at J1.2 (D0): now also U3.2 (A0); no longer U3.15 (I2b)
- net at J1.8 (D6): now also U3.8 (A6); no longer U3.2 (I0a)
- net at J1.7 (D5): now also U3.7 (A5); no longer U3.4 (I1a)
- net at J1.5 (D3): now also U3.5 (A3); no longer U3.8 (I3a)
- net at J5.4 (D2): now also U7.4 (A2); no longer U7.11 (I0b)
- net at J5.3 (D1): now also U7.3 (A1); no longer U7.13 (I1b)
- net at J5.2 (D0): now also U7.2 (A0); no longer U7.15 (I2b)
- net at J5.8 (D6): now also U7.8 (A6); no longer U7.2 (I0a)
- net at J5.7 (D5): now also U7.7 (A5); no longer U7.4 (I1a)
- net at J5.5 (D3): now also U7.5 (A3); no longer U7.8 (I3a)
- net at J4.2 (D0): now also U6.2 (A0); no longer U6.15 (I2b)
- net at J4.3 (D1): now also U6.3 (A1); no longer U6.13 (I1b)
- net at J4.4 (D2): now also U6.4 (A2); no longer U6.11 (I0b)
- net at J4.5 (D3): now also U6.5 (A3); no longer U6.8 (I3a)
- net at J4.7 (D5): now also U6.7 (A5); no longer U6.4 (I1a)
- net at J4.8 (D6): now also U6.8 (A6); no longer U6.2 (I0a)
- net at J7.2 (D0): now also U9.2 (A0); no longer U9.15 (I2b)
- net at J7.3 (D1): now also U9.3 (A1); no longer U9.13 (I1b)
- net at J7.4 (D2): now also U9.4 (A2); no longer U9.11 (I0b)
- net at J7.5 (D3): now also U9.5 (A3); no longer U9.8 (I3a)
- net at J7.7 (D5): now also U9.7 (A5); no longer U9.4 (I1a)
- net at J7.8 (D6): now also U9.8 (A6); no longer U9.2 (I0a)
- net at J3.2 (D0): now also U5.2 (A0); no longer U5.15 (I2b)
- net at J3.3 (D1): now also U5.3 (A1); no longer U5.13 (I1b)
- net at J3.4 (D2): now also U5.4 (A2); no longer U5.11 (I0b)
- net at J3.5 (D3): now also U5.5 (A3); no longer U5.8 (I3a)
- net at J3.7 (D5): now also U5.7 (A5); no longer U5.4 (I1a)
- net at J3.8 (D6): now also U5.8 (A6); no longer U5.2 (I0a)
- new net: J6.9 (D7), U8.9 (A7)
- new net: J2.9 (D7), U4.9 (A7)
- new net: J8.9 (D7), U10.9 (A7)
- new net: J1.9 (D7), U3.9 (A7)
- new net: J5.9 (D7), U7.9 (A7)
- new net: J4.9 (D7), U6.9 (A7)
- new net: J7.9 (D7), U9.9 (A7)
- new net: J3.9 (D7), U5.9 (A7)
- new net ~{EN}: U1.4 (CTRL_{0}), U10.19 (G2), U2.4 (~{E1}), U2.5 (~{E2}), U3.19 (G2), U4.19 (G2), U5.19 (G2), U6.19 (G2), U7.19 (G2), U8.19 (G2), U9.19 (G2)
- now unconnected: U1.12 (GND), U1.14 (GND)
