File: v1/kicad/sp_register/sp_register.kicad_pcb (KiCad board)
At the start: 2 copper layers, 101.5 x 66.5 mm, 12 parts, among them J1 OP_{out}, U1 LNCPU Type B Connector, U2 74LS169, U3 74LS169, U4 74HCT541, U5 74HCT00

Commit message: readapt designs for BR, SP, SR, ALU
Connections:
- J1 pad 10: /GND -> /VCC
Routing:
- net /VCC: track 247.5 -> 258.4 mm, vias 4 -> 6
- net /GND: track 308.1 -> 301.9 mm
Changed lines of the file:
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@@
 			(layers "*.Cu" "*.Mask")
 			(remove_unused_layers no)
-			(net 1 "/GND")
-			(pinfunction "GND")
+			(net 2 "/VCC")
+			(pinfunction "VCC")
 			(pintype "passive")
 		)
@@
 	)
 	(segment
-		(start 132.16 79.885)
-		(end 132.16 73.6582)
-		(width 0.8)
-		(layer "B.Cu")
-		(net 1)
-	)
-	(segment
 		(start 176.7365 61.6165)
 		(end 177.6247 62.5046)
@@
 		(start 159.8067 73.3217)
 		(end 160.8417 74.3567)
+		(width 0.8)
+		(layer "F.Cu")
+		(net 2)
+	)
+	(segment
+		(start 124.54 76.788)
+		(end 124.46 76.708)
+		(width 0.8)
+		(layer "F.Cu")
+		(net 2)
+	)
+	(segment
+		(start 132.16 76.788)
+		(end 124.54 76.788)
 		(width 0.8)
 		(layer "F.Cu")
@@
 	)
 	(via
+		(at 124.2242 76.708)
+		(size 1.6)
+		(drill 0.8)
+		(layers "F.Cu" "B.Cu")
+		(net 2)
+	)
+	(via
 		(at 197.4846 74.3567)
 		(size 1.6)
@@
 		(net 2)
 	)
+	(via
+		(at 132.16 76.788)
+		(size 1.6)
+		(drill 0.8)
+		(layers "F.Cu" "B.Cu")
+		(net 2)
+	)
 	(segment
 		(start 196.04 43)
@@
 	)
 	(segment
+		(start 132.16 79.885)
+		(end 132.16 76.788)
+		(width 0.8)
+		(layer "B.Cu")
+		(net 2)
+	)
+	(segment
 		(start 150.74 41.8)
 		(end 150.74 39.8)
@@
 	(segment
 		(start 124.2242 84.7484)
-		(end 124.2242 67.7248)
+		(end 124.2242 76.708)
 		(width 0.8)
 		(layer "B.Cu")
@@
 	)
 	(segment
+		(start 132.16 76.788)
+		(end 132.08 76.708)
+		(width 0.8)
+		(layer "B.Cu")
+		(net 2)
+	)
+	(segment
 		(start 114.4576 85.9726)
 		(end 114.45 85.965)
@@
 		(width 0.8)
 		(layer "B.Cu")
+		(net 2)
+	)
+	(segment
+		(start 124.2242 76.708)
+		(end 124.2242 67.7248)
+		(width 0.8)
+		(layer "B.Cu")
