File: v1/kicad/flags/FlagsCtrl.kicad_sch (KiCad schematic)
At the start: 7 parts, among them U1 74LS32, U2 74LS08, U3 74LS32, U4 74AHC04, U5 74LS32, U6 74LS157, U7 74LS157

Commit message: partial on kicad flags
Parts:
- added C10, C11, C5, C6, C7, C8, C9: 100n, Capacitor_THT:C_Disc_D5.0mm_W2.5mm_P2.50mm, symbol Device:C
- U10: renamed from U4; value 74AHC04 -> 74LS04; symbol 74xx:74AHC04 -> 74xx:74LS04
- renumbered U6 to U11, U7 to U12, U5 to U13, U2 to U3, U3 to U5, U1 to U9
Connections:
- net GND: now also U10.7 (GND), U13.7 (GND), U3.7 (GND), U5.7 (GND), U9.7 (GND), C10.1, C11.1, C5.2, C6.2, C7.1, C8.1, C9.1; no longer U10.14 (VCC), U13.14 (VCC), U3.14 (VCC), U5.14 (VCC), U9.14 (VCC)
- net VCC: now also U10.14 (VCC), U13.14 (VCC), U3.14 (VCC), U5.14 (VCC), U9.14 (VCC), C10.2, C11.2, C5.1, C6.1, C7.2, C8.2, C9.2; no longer U10.7 (GND), U13.7 (GND), U3.7 (GND), U5.7 (GND), U9.7 (GND)
- net ~{CZ_{in}} renamed ~{NZ_{in}}
Other:
- moved on the sheet: U10B, U10E, U10F, U10G, U11, U12, U13A, U13B, U13C, U13D, U13E, U3B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
