File: v1/kicad/flags/flags.kicad_sch (KiCad schematic)
At the start: 8 parts, among them J1 LNCPU_FLAGS_Socket, U10 74LS08, U11 74HC173, U12 74LS244, U2 74LS08, U3 74LS32, U8 LNCPU Type B Connector, U9 74HC74

Commit message: partial on kicad flags
Parts:
- added C1, C2: 220n, Capacitor_THT:C_Disc_D5.0mm_W2.5mm_P2.50mm, symbol Device:C
- added C12: C_Polarized, Capacitor_THT:CP_Radial_D5.0mm_P2.00mm, symbol Device:C_Polarized
- added C13: C_Polarized, lncpu:CP_Radial_D4.0mm_P2.00mm-Large-Holes, symbol Device:C_Polarized
- added C3, C4: 100n, Capacitor_THT:C_Disc_D5.0mm_W2.5mm_P2.50mm, symbol Device:C
- added unit 4 of U2
- added unit 3 of U2
- J1: value LNCPU_FLAGS_Socket -> LNCPU_FLAGS_Connector; footprint Connector_PinSocket_2.54mm:PinSocket_1x04_P2.54mm_Vertical -> Connector_PinSocket_2.54mm:PinSocket_1x06_P2.54mm_Vertical
- U1: renamed from U8; value LNCPU Type B Connector -> LNCPU Type B Header; symbol lncpu:LNCPU_Type_B_Connector -> lncpu:LNCPU_Type_B_Header
- U4: renamed from U11; value 74HC173 -> 74HCT173; symbol 74xx:74HC173 -> 74xx:74HCT173
- U6: renamed from U9; value 74HC74 -> 74HCT74; symbol 74xx:74HC74 -> 74xx:74HCT74
- U8: renamed from U12; value 74LS244 -> 74HCT541; symbol 74xx:74LS244 -> 74xx:74HCT541
- renumbered U10 to U2, U2 to U3, U3 to U5
Connections:
- net DBUS0: now also U1.3 (DBUS_{0}); no longer U1.4 (DBUS_{0})
- net DBUS1: now also U1.5 (DBUS_{1}), U8.17 (Y1); no longer U1.6 (DBUS_{1}), U8.16 (O1a)
- net DBUS2: now also U1.7 (DBUS_{2}), U8.16 (Y2); no longer U1.8 (DBUS_{2}), U8.14 (O2a)
- net DBUS3: now also U1.9 (DBUS_{3}), U8.15 (Y3); no longer U1.10 (DBUS_{3}), U8.12 (O3a)
- net DBUS4: now also U1.11 (DBUS_{4}), U8.14 (Y4); no longer U1.12 (DBUS_{4}), U8.9 (O0b)
- net DBUS5: now also U1.13 (DBUS_{5}), U8.13 (Y5); no longer U1.14 (DBUS_{5}), U8.7 (O1b)
- net DBUS6: now also U1.15 (DBUS_{6}), U8.12 (Y6); no longer U1.16 (DBUS_{6}), U8.5 (O2b)
- net DBUS7: now also U1.17 (DBUS_{7}), U8.11 (Y7); no longer U1.18 (DBUS_{7}), U8.3 (O3b)
- net FlagsCtrl/ALU_{Cin}: now also U1.14 (CTRL_{5}); no longer U1.13 (CTRL_{5})
- net FlagsCtrl/MODE_{0}: now also U1.8 (CTRL_{2}); no longer U1.7 (CTRL_{2})
- net FlagsCtrl/MODE_{1}: now also U1.10 (CTRL_{3}); no longer U1.9 (CTRL_{3})
- net FlagsCtrl/MODE_{2}: now also U1.12 (CTRL_{4}); no longer U1.11 (CTRL_{4})
- net GND: now also J1.1 (GND), U1.18 (GND), U1.23 (GND), U8.6 (A4), U8.7 (A5), U8.8 (A6), U8.9 (A7), C1.2, C12.2, C13.2, C2.2, C3.2, C4.2, U2.10, U2.12, U2.13, U2.9; no longer U1.17 (GND), U1.20 (GND), U2.10, U2.12, U2.13, U2.9, U8.11 (I0b), U8.13 (I1b), U8.15 (I2b), U8.17 (I3b)
- net VCC: now also J1.6 (VCC), C1.1, C12.1, C13.1, C2.1, C3.1, C4.1
- net at U4.10 (E2), U8.1 (G1): now also U1.4 (CTRL_{0}); no longer U1.3 (CTRL_{0})
- net at U8.19 (G2): now also U1.6 (CTRL_{1}); no longer U1.5 (CTRL_{1})
- net at U2.5, U6.5 (Q), U8.2 (A0): now also J1.2 (C); no longer J1.1 (C)
- net at U3.12, U6.9 (Q): now also J1.5 (I), U8.5 (A3); no longer J1.4 (I), U8.8 (I3a)
- net FlagsCtrl/~{CZ_{in}} renamed FlagsCtrl/~{NZ_{in}}
- new net: J1.3 (Z), U4.3 (Q0), U8.3 (A1)
- new net: J1.4 (N), U4.4 (Q1), U8.4 (A2)
Other:
- sheet FlagsCtrl ports: added ~{NZ_{in}}; removed ~{CZ_{in}}
- moved on the sheet: U1, U2E
